Commit message: Controllers for wrist and gripper not used. Topics created for controlling wrist and gripper if needed.

File: src/cepheus_robot/model/cepheus.urdf (robot description, URDF)
Before this commit: robot cepheus, 6 links, 5 joints
Joints:
- joint left_wrist: limit lower=-1.570796327 upper=1.570796327 effort=1 velocity=10 -> lower=20 upper=150 effort=1 velocity=10

Commit message: 1)Left elbow limit calculated again and corrected in urdf and launch. 2)Movement of left arm transformed to callback -> works ok. Action added: left wrist trajectory movement. 3)Topic created that controls the action of the left gripper (open - close). Close not correct-> needs improvement and re-init in left fsr controller

File: src/cepheus_robot/model/cepheus.urdf (robot description, URDF)
Before this commit: robot cepheus, 6 links, 5 joints
Joints:
- joint left_elbow: limit lower=-3.14 upper=1.5 effort=2 velocity=20 -> lower=-3.14 upper=1.75 effort=2 velocity=20

Commit message: Started to work on inverse kinematics for left arm. Trying to grip object with fixed pos and close to cepheus. Nikos calculated the equation giving the set point for each joint. Code added. NEEDS TESTING AND MODIFICATIONS.

File: src/cepheus_robot/model/cepheus.urdf (robot description, URDF)
Before this commit: robot cepheus, 6 links, 5 joints
Links:
- link cepheus: geometry collision cylinder length=0.43 radius=0.2; visual mesh filename=file://cepheus_robot/meshes/cepheus.STL
- link reaction_wheel: geometry visual mesh filename=file://cepheus_robot/meshes/reaction_wheel.STL

Commit message: Functions for right arm init added. Problem with reading hall sensors

File: src/cepheus_robot/model/cepheus.urdf (robot description, URDF)
Before this commit: robot cepheus, 6 links, 5 joints
Links:
- added link right_arm, mass 0.07974; collision box size=0.13 0.02 0.02
- added link right_forearm, mass 0.06392; collision box size=0.13 0.025 0.025
Joints:
- added joint right_elbow: type revolute, parent right_arm, child right_forearm, origin xyz=0.18120 0.01176 -0.002 rpy=0 0 0, axis 0 0 1, limit lower=3.14 upper=-1.75 effort=2 velocity=20
- added joint right_shoulder: type revolute, parent cepheus, child right_arm, origin xyz=0.17271 -0.091404 0.05875 rpy=0 0 0, axis 0 0 1, limit lower=0.86 upper=-2.54 effort=20 velocity=20

Commit message: Small problem with right hand init solved. Arm limits have to be updated in the .yaml file too

File: src/cepheus_robot/model/cepheus.urdf (robot description, URDF)
Before this commit: robot cepheus, 8 links, 7 joints
Joints:
- joint right_elbow: limit lower=3.14 upper=-1.75 effort=2 velocity=20 -> lower=-1.75 upper=3.14 effort=2 velocity=20
- joint right_shoulder: limit lower=0.86 upper=-2.54 effort=20 velocity=20 -> lower=-2.54 upper=0.86 effort=20 velocity=20

Commit message: Inverse kinematics ( for right arm) BUG is corrected. It seems to work fine. I need to copy the code for the left arm inv kin too. Init in right arm seems ok too

File: src/cepheus_robot/model/cepheus.urdf (robot description, URDF)
Before this commit: robot cepheus, 8 links, 7 joints
Joints:
- joint right_elbow: limit lower=-1.75 upper=3.14 effort=2 velocity=20 -> lower=-1.575 upper=3.14 effort=2 velocity=20
- joint right_shoulder: limit lower=-2.54 upper=0.86 effort=20 velocity=20 -> lower=-2.453 upper=0.86 effort=20 velocity=20

Commit message: No more experiments! Some cleaning

File: src/cepheus_robot/model/cepheus.urdf (robot description, URDF)
Before this commit: robot cepheus, 8 links, 7 joints
Joints:
- joint right_elbow: limit lower=-1.575 upper=3.14 effort=2 velocity=20 -> lower=-1.6231 upper=3.14 effort=2 velocity=20

Commit message: Init changes for 2020 tests

File: src/cepheus_robot/model/cepheus.urdf (robot description, URDF)
Before this commit: robot cepheus, 8 links, 7 joints
Joints:
- joint left_shoulder: limit lower=-0.86 upper=2.54 effort=20 velocity=20 -> lower=-0.86 upper=3.154 effort=20 velocity=20

Commit message: Add services to set position offsets for motors

File: src/cepheus_robot/model/cepheus.urdf (robot description, URDF)
Before this commit: robot cepheus, 8 links, 7 joints
Joints:
- joint left_elbow: limit lower=-3.14 upper=1.75 effort=2 velocity=20 -> lower=-0.92 upper=2.33 effort=2 velocity=20
- joint left_shoulder: limit lower=-0.86 upper=3.154 effort=20 velocity=20 -> lower=-1.34 upper=1.34 effort=20 velocity=20
- joint right_elbow: limit lower=-1.6231 upper=3.14 effort=2 velocity=20 -> lower=0.00 upper=1.65 effort=2 velocity=20

Commit message: Limit tweaks

File: src/cepheus_robot/model/cepheus.urdf (robot description, URDF)
Before this commit: robot cepheus, 8 links, 7 joints
Joints:
- joint left_shoulder: limit lower=-1.34 upper=1.34 effort=20 velocity=20 -> lower=-1.33 upper=1.33 effort=20 velocity=20
- joint right_elbow: limit lower=0.00 upper=1.65 effort=2 velocity=20 -> lower=0.00 upper=1.80 effort=2 velocity=20

Commit message: Complete init, add phase space track three objects

File: src/cepheus_robot/model/cepheus.urdf (robot description, URDF)
Before this commit: robot cepheus, 8 links, 7 joints
Links:
- removed link left_finger
- removed link left_grip
Joints:
- removed joint left_finger_joint
- removed joint left_wrist
